File: PCB/Tamagotchi.kicad_sch (KiCad schematic)
At the start: 7 parts, among them J1 Conn_01x02_Pin, SW1 C13828, SW2 C13828, SW3 C13828, U2 HS96L03W2C03, U3 XIAO-ESP32-C6-SMD

Commit message: Add files via upload
Parts:
- renumbered BUZZER1 to PASSIVEBUZZER1
Changed lines of the file:
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@@
 		(dnp no)
 		(fields_autoplaced yes)
-		(property "Reference" "BUZZER1"
+		(property "Reference" "PASSIVEBUZZER1"
 			(at 209.55 110.4899 0)
 			(effects
@@
 			(project ""
 				(path "/dda21022-0147-4ac7-b935-5203eac868ff"
-					(reference "BUZZER1")
+					(reference "PASSIVEBUZZER1")
 					(unit 1)
 				)
